File: HackPad.kicad_pcb (KiCad board)
At the start: 2 copper layers, 7 parts, among them SW1 SW_Push, SW2 SW_Push, SW3 SW_Push, SW5 RotaryEncoder_Switch, U1 XIAO-RP2040-DIP

Commit message: teto board
Parts:
- added G***: LOGO, LOGO, F.Cu at (93.8, 49.2)
- moved D2 4.65 mm to (60.0, 68.5)
- moved D1 4.65 mm to (111.7, 68.5)
Routing:
- net GPIO1: track 0.00 -> 41.2 mm, vias 0 -> 2
- net GND: track 181.3 -> 144.2 mm
- net ENC_B: track 0.00 -> 33.8 mm, vias 0 -> 2
- net GPIO2: track 0.00 -> 29.5 mm, vias 0 -> 1
- net ENC_A: track 0.00 -> 23.5 mm
- net GPIO4: track 0.00 -> 22.5 mm, vias 0 -> 1
- net Net-(D1-DOUT): track 66.2 -> 57.5 mm
- net +5V: track 103.3 -> 103.0 mm, vias 3 -> 1
Other:
- board outline added: 61.2 x 46.2 mm
- board text added: "Nat3z 2025"
- board text added: "teto board"
- board text added: "{dblquote}I am definite and real!{dblquote}"
